File: SuniderPra/Controller.brd (EAGLE design)
At the start: 60 x 50 mm, 7 parts, among them X1 B6B-XH-2

Commit message: Add files via upload
Parts:
- added X2: B7B-XH-2, con-JST XH:B7B-XH-A
- X1: value B6B-XH-2 -> B2B-XH-2; device con-JST XH:B6B-XH-A -> con-JST XH:B2B-XH-A
- moved X1 17.4 mm to (50.0, 39.0)
Connections:
- new net +9V: X1.1, X2.6
- net +3V3: now also X2.5; no longer X1.5
- net GND: now also X1.2, X2.7; no longer X1.6
- net N$2: now also X2.3; no longer X1.3
- net N$3: now also X2.2; no longer X1.2
- net N$4: now also X2.1; no longer X1.1
- net N$5: now also X2.4; no longer X1.4
Routing:
- net +9V: track 0.00 -> 26.8 mm, vias 0 -> 1
- net N$4: track 38.7 -> 45.0 mm
- net N$2: track 28.7 -> 26.8 mm
- net N$3: track 57.0 -> 56.1 mm
- net N$5: track 28.2 -> 27.4 mm
Changed lines of the file:
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@@
 <classes>
 <class number="0" name="default" width="0" drill="0">
+<clearance class="0" value="0.508"/>
 </class>
 </classes>
@@
 <attribute name="VALUE" x="32.1388" y="30.934" size="1.27" layer="27" ratio="10" rot="R90"/>
 </element>
-<element name="X1" library="con-JST XH" package="B6B-XH-A" value="B6B-XH-2" x="33.64" y="44.9" smashed="yes" rot="R180">
-<attribute name="NAME" x="24.342" y="44.9" size="1.016" layer="25" rot="R90" align="bottom-center"/>
-<attribute name="VALUE" x="27.39" y="43.63" size="1.016" layer="27" rot="R180" align="bottom-right"/>
-</element>
 <element name="LED1" library="led" library_urn="urn:adsk.eagle:library:259" package="LED3MM" package3d_urn="urn:adsk.eagle:package:15797/1" value="" x="36" y="23" smashed="yes" rot="R270">
 <attribute name="NAME" x="33.905" y="19.381" size="1.27" layer="25" ratio="10"/>
@@
 </element>
 <element name="JOY1" library="JOYSTICK" package="JOY" value="JOY" x="14" y="18" smashed="yes"/>
+<element name="X2" library="con-JST XH" package="B7B-XH-A" value="B7B-XH-2" x="34" y="45" smashed="yes" rot="R180">
+<attribute name="NAME" x="23.452" y="45" size="1.016" layer="25" rot="R90" align="bottom-center"/>
+<attribute name="VALUE" x="26.5" y="43.73" size="1.016" layer="27" rot="R180" align="bottom-right"/>
+</element>
+<element name="X1" library="con-JST XH" package="B2B-XH-A" value="B2B-XH-2" x="50" y="39" smashed="yes" rot="R180">
+<attribute name="NAME" x="45.702" y="39" size="1.016" layer="25" rot="R90" align="bottom-center"/>
+<attribute name="VALUE" x="48.75" y="37.73" size="1.016" layer="27" rot="R180" align="bottom-right"/>
+</element>
 </elements>
 <signals>
 <signal name="GND">
-<contactref element="X1" pad="6"/>
 <contactref element="POT1" pad="P$1"/>
 <polygon width="0.254" layer="16">
@@
 <contactref element="C1" pad="1"/>
 <contactref element="JOY1" pad="P$1"/>
+<contactref element="X2" pad="7"/>
+<contactref element="X1" pad="2"/>
 </signal>
 <signal name="+3V3">
-<contactref element="X1" pad="5"/>
 <contactref element="R1" pad="2"/>
 <contactref element="POT1" pad="P$2"/>
@@
 <wire x1="39" y1="35.54" x2="39" y2="38.53999375" width="1.016" layer="1"/>
 <wire x1="39" y1="38.53999375" x2="37.39" y2="40.1499875" width="1.016" layer="1"/>
-<wire x1="37.39" y1="44.9" x2="37.39" y2="40.1499875" width="1.016" layer="1"/>
 <wire x1="39" y1="35.54" x2="40.55" y2="35.54" width="0.508" layer="1"/>
 <wire x1="45.41" y1="30.68" x2="40.55" y2="35.54" width="0.508" layer="1"/>
@@
 <wire x1="16.5" y1="43" x2="21.96" y2="37.54" width="0.508" layer="1"/>
 <wire x1="21.96" y1="37.54" x2="33.09" y2="37.54" width="0.508" layer="1"/>
+<contactref element="X2" pad="5"/>
+<wire x1="37.39" y1="40.1499875" x2="36.5" y2="41.0399875" width="1.016" layer="1"/>
+<wire x1="36.5" y1="41.0399875" x2="36.5" y2="45" width="1.016" layer="1"/>
 </signal>
 <signal name="N$2">
-<contactref element="X1" pad="3"/>
 <contactref element="JOY1" pad="P$4"/>
-<wire x1="32.39" y1="44.9" x2="32.39" y2="42.9" width="0.508" layer="1"/>
-<wire x1="32.39" y1="42.9" x2="30.49" y2="41" width="0.508" layer="1"/>
-<wire x1="30.49" y1="41" x2="26" y2="41" width="0.508" layer="1"/>
 <wire x1="11.5" y1="44.5" x2="11.5" y2="43" width="0.508" layer="1"/>
-<wire x1="26" y1="41" x2="20" y2="47" width="0.508" layer="1"/>
-<wire x1="20" y1="47" x2="14" y2="47" width="0.508" layer="1"/>
-<wire x1="14" y1="47" x2="11.5" y2="44.5" width="0.508" layer="1"/>
+<wire x1="24.7" y1="41.6" x2="24.65" y2="41.65" width="0.508" layer="1"/>
+<wire x1="24.65" y1="41.65" x2="19.7" y2="46.6" width="0.508" layer="1"/>
+<wire x1="19.7" y1="46.6" x2="13.6" y2="46.6" width="0.508" layer="1"/>
+<wire x1="13.6" y1="46.6" x2="11.5" y2="44.5" width="0.508" layer="1"/>
+<contactref element="X2" pad="3"/>
+<wire x1="24.65" y1="41.65" x2="29.65" y2="41.65" width="0.508" layer="1"/>
+<wire x1="31.5" y1="43.5" x2="31.5" y2="45" width="0.508" layer="1"/>
+<wire x1="29.65" y1="41.65" x2="31.5" y2="43.5" width="0.508" layer="1"/>
 </signal>
 <signal name="N$3">
-<contactref element="X1" pad="2"/>
 <contactref element="R1" pad="1"/>
 <contactref element="JOY1" pad="P$5"/>
-<wire x1="29.89" y1="44.9" x2="29.89" y2="43.89" width="0.508" layer="1"/>
-<wire x1="29.89" y1="43.89" x2="29" y2="43" width="0.508" layer="1"/>
-<wire x1="29" y1="43" x2="26" y2="43" width="0.508" layer="1"/>
-<wire x1="21" y1="48" x2="12" y2="48" width="0.508" layer="1"/>
+<wire x1="20.6" y1="48" x2="12" y2="48" width="0.508" layer="1"/>
 <wire x1="12" y1="48" x2="8.9" y2="44.9" width="0.508" layer="1"/>
 <wire x1="8.9" y1="44.9" x2="8.9" y2="43" width="0.508" layer="1"/>
-<wire x1="26" y1="43" x2="21" y2="48" width="0.508" layer="1"/>
+<wire x1="20.6" y1="48" x2="25.6" y2="43" width="0.508" layer="1"/>
 <wire x1="8.9" y1="43" x2="8.9" y2="41.93" width="0.508" layer="1"/>
 <wire x1="8.9" y1="41.93" x2="22.42" y2="28.41" width="0.508" layer="1"/>
 <wire x1="22.42" y1="28.41" x2="31.58" y2="28.41" width="0.508" layer="1"/>
+<contactref element="X2" pad="2"/>
+<wire x1="25.6" y1="43" x2="28" y2="43" width="0.508" layer="1"/>
+<wire x1="28" y1="43" x2="29" y2="44" width="0.508" layer="1"/>
+<wire x1="29" y1="44" x2="29" y2="45" width="0.508" layer="1"/>
 </signal>
 <signal name="N$4">
-<contactref element="X1" pad="1"/>
 <contactref element="POT1" pad="P$3"/>
 <wire x1="28.39" y1="47" x2="28.39" y2="46.9" width="0.508" layer="1"/>
-<wire x1="28.39" y1="46.9" x2="27.39" y2="45.9" width="0.508" layer="1"/>
-<wire x1="27.39" y1="44.9" x2="27.39" y2="45.9" width="0.508" layer="1"/>
-<wire x1="28.39" y1="47" x2="40" y2="47" width="0.508" layer="1"/>
-<wire x1="50.31" y1="36.69" x2="50.31" y2="26.68" width="0.508" layer="1"/>
-<wire x1="40" y1="47" x2="50.31" y2="36.69" width="0.508" layer="1"/>
+<wire x1="27.39" y1="45.9" x2="28.39" y2="46.9" width="0.508" layer="1"/>
+<wire x1="28.39" y1="47" x2="46" y2="47" width="0.508" layer="1"/>
+<wire x1="53.31" y1="39.69" x2="53.31" y2="29.68" width="0.508" layer="1"/>
+<wire x1="53.31" y1="29.68" x2="50.31" y2="26.68" width="0.508" layer="1"/>
+<wire x1="46" y1="47" x2="53.31" y2="39.69" width="0.508" layer="1"/>
+<contactref element="X2" pad="1"/>
+<wire x1="26.5" y1="45" x2="27.39" y2="45.89" width="0.508" layer="1"/>
+<wire x1="27.39" y1="45.89" x2="27.39" y2="45.9" width="0.508" layer="1"/>
 </signal>
 <signal name="N$15">
@@
 </signal>
 <signal name="N$5">
-<contactref element="X1" pad="4"/>
 <contactref element="JOY1" pad="P$3"/>
-<wire x1="34.89" y1="44.9" x2="34.89" y2="41.9" width="0.508" layer="1"/>
-<wire x1="32.99" y1="40" x2="34.89" y2="41.9" width="0.508" layer="1"/>
 <wire x1="14" y1="43" x2="14" y2="44" width="0.508" layer="1"/>
 <wire x1="14" y1="44" x2="15" y2="45" width="0.508" layer="1"/>
-<wire x1="15" y1="45" x2="20" y2="45" width="0.508" layer="1"/>
-<wire x1="20" y1="45" x2="25" y2="40" width="0.508" layer="1"/>
-<wire x1="25" y1="40" x2="32.99" y2="40" width="0.508" layer="1"/>
+<wire x1="15" y1="45" x2="19.3" y2="45" width="0.508" layer="1"/>
+<wire x1="19.3" y1="45" x2="24.15" y2="40.15" width="0.508" layer="1"/>
+<contactref element="X2" pad="4"/>
+<wire x1="24.15" y1="40.15" x2="24.3" y2="40" width="0.508" layer="1"/>
+<wire x1="24.15" y1="40.15" x2="32.15" y2="40.15" width="0.508" layer="1"/>
+<wire x1="34" y1="42" x2="34" y2="45" width="0.508" layer="1"/>
+<wire x1="32.15" y1="40.15" x2="34" y2="42" width="0.508" layer="1"/>
+</signal>
+<signal name="+9V">
+<contactref element="X2" pad="6"/>
+<contactref element="X1" pad="1"/>
+<wire x1="48.75" y1="39" x2="43" y2="39" width="1.8" layer="1"/>
+<wire x1="39" y1="43" x2="39" y2="45" width="1.8" layer="1"/>
+<wire x1="43" y1="39" x2="41" y2="41" width="1.8" layer="1"/>
+<wire x1="41" y1="41" x2="39" y2="43" width="1.8" layer="1"/>
+<wire x1="48.75" y1="39" x2="43" y2="39" width="1.8" layer="16"/>
+<wire x1="43" y1="39" x2="41" y2="41" width="1.8" layer="16"/>
+<wire x1="41" y1="41" x2="39" y2="43" width="1.8" layer="16"/>
+<wire x1="39" y1="43" x2="39" y2="45" width="1.8" layer="16"/>
+<via x="41" y="41" extent="1-16" drill="0.35"/>
 </signal>
 </signals>
