File: SuniderPra/Controller.sch (EAGLE design)
At the start: 7 parts, among them X1 B6B-XH-2

Commit message: Add files via upload
Parts:
- added X2: B7B-XH-2, con-JST XH:B7B-XH-2
- X1: value B6B-XH-2 -> B2B-XH-2; device con-JST XH:B6B-XH-2 -> con-JST XH:B2B-XH-2
Connections:
- new net +9V: X1.1, X2.6
- net +3V3: now also X2.5; no longer X1.5
- net GND: now also X1.2, X2.7; no longer X1.6
- net N$2: now also X2.3; no longer X1.3
- net N$3: now also X2.2; no longer X1.2
- net N$4: now also X2.1; no longer X1.1
- net N$5: now also X2.4; no longer X1.4
Changed lines of the file:
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@@
 <classes>
 <class number="0" name="default" width="0" drill="0">
+<clearance class="0" value="0.508"/>
 </class>
 </classes>
 <parts>
-<part name="X1" library="con-JST XH" deviceset="B6B-XH" device="-2"/>
 <part name="POT1" library="potentiometer" deviceset="POTENTIOMETER" device=""/>
 <part name="SUPPLY1" library="supply2" library_urn="urn:adsk.eagle:library:372" deviceset="GND" device=""/>
@@
 <part name="SUPPLY4" library="supply2" library_urn="urn:adsk.eagle:library:372" deviceset="GND" device=""/>
 <part name="JOY1" library="JOYSTICK" deviceset="JOY" device=""/>
+<part name="X2" library="con-JST XH" deviceset="B7B-XH" device="-2"/>
+<part name="SUPPLY5" library="supply2" library_urn="urn:adsk.eagle:library:372" deviceset="+9V" device=""/>
+<part name="SUPPLY6" library="supply2" library_urn="urn:adsk.eagle:library:372" deviceset="+9V" device=""/>
+<part name="X1" library="con-JST XH" deviceset="B2B-XH" device="-2"/>
+<part name="SUPPLY7" library="supply2" library_urn="urn:adsk.eagle:library:372" deviceset="GND" device=""/>
 </parts>
 <sheets>
@@
 </plain>
 <instances>
-<instance part="X1" gate="G$1" x="28" y="11" smashed="yes" rot="R180">
-<attribute name="VALUE" x="29.27" y="23.7" size="1.778" layer="96" rot="R180"/>
-<attribute name="NAME" x="29.27" y="2.618" size="1.778" layer="95" rot="R180"/>
-</instance>
 <instance part="POT1" gate="G$1" x="16" y="31" smashed="yes" rot="R270"/>
-<instance part="SUPPLY1" gate="GND" x="12" y="6" smashed="yes" rot="R270">
-<attribute name="VALUE" x="8.825" y="7.905" size="1.778" layer="96" rot="R270"/>
+<instance part="SUPPLY1" gate="GND" x="13" y="3" smashed="yes" rot="R270">
+<attribute name="VALUE" x="9.825" y="4.905" size="1.778" layer="96" rot="R270"/>
 </instance>
 <instance part="+3V1" gate="G$1" x="12" y="9" smashed="yes" rot="R90">
-<attribute name="VALUE" x="17.08" y="6.46" size="1.778" layer="96" rot="R180"/>
+<attribute name="VALUE" x="10.08" y="9.46" size="1.778" layer="96" rot="R180"/>
 </instance>
 <instance part="+3V2" gate="G$1" x="-1" y="9" smashed="yes" rot="R270">
@@
 </instance>
 <instance part="JOY1" gate="G$1" x="-25" y="11" smashed="yes" rot="R270"/>
+<instance part="X2" gate="G$1" x="28" y="11" smashed="yes" rot="R180">
+<attribute name="VALUE" x="29.27" y="23.7" size="1.778" layer="96" rot="R180"/>
+<attribute name="NAME" x="29.27" y="0.078" size="1.778" layer="95" rot="R180"/>
+</instance>
+<instance part="SUPPLY5" gate="G$1" x="12" y="6" smashed="yes" rot="R90">
+<attribute name="VALUE" x="8.905" y="6.825" size="1.778" layer="96" rot="R180"/>
+</instance>
+<instance part="SUPPLY6" gate="G$1" x="-28" y="34" smashed="yes" rot="R270">
+<attribute name="VALUE" x="-24.825" y="35.905" size="1.778" layer="96" rot="R270"/>
+</instance>
+<instance part="X1" gate="G$1" x="-43" y="37" smashed="yes">
+<attribute name="VALUE" x="-44.27" y="29.38" size="1.778" layer="96"/>
+<attribute name="NAME" x="-44.27" y="40.302" size="1.778" layer="95"/>
+</instance>
+<instance part="SUPPLY7" gate="GND" x="-27" y="37" smashed="yes" rot="R90">
+<attribute name="VALUE" x="-23.825" y="35.095" size="1.778" layer="96" rot="R90"/>
+</instance>
 </instances>
 <busses>
@@
 <net name="GND" class="0">
 <segment>
-<wire x1="19" y1="6" x2="14.54" y2="6" width="0.1524" layer="91"/>
-<pinref part="SUPPLY1" gate="GND" pin="GND"/>
-<pinref part="X1" gate="G$1" pin="6"/>
-<wire x1="19" y1="6" x2="19" y2="5.92" width="0.1524" layer="91"/>
-<wire x1="19" y1="5.92" x2="20.38" y2="5.92" width="0.1524" layer="91"/>
-</segment>
-<segment>
 <pinref part="POT1" gate="G$1" pin="P$1"/>
 <wire x1="29.46" y1="31" x2="26" y2="31" width="0.1524" layer="91"/>
@@
 <pinref part="JOY1" gate="G$1" pin="GND"/>
 </segment>
+<segment>
+<wire x1="15.54" y1="3" x2="20" y2="3" width="0.1524" layer="91"/>
+<pinref part="X2" gate="G$1" pin="7"/>
+<wire x1="20" y1="3" x2="20" y2="3.38" width="0.1524" layer="91"/>
+<wire x1="20" y1="3.38" x2="20.38" y2="3.38" width="0.1524" layer="91"/>
+<pinref part="SUPPLY1" gate="GND" pin="GND"/>
+</segment>
+<segment>
+<wire x1="-29.54" y1="37" x2="-35.38" y2="37" width="0.1524" layer="91"/>
+<pinref part="X1" gate="G$1" pin="2"/>
+<pinref part="SUPPLY7" gate="GND" pin="GND"/>
+</segment>
 </net>
 <net name="+3V3" class="0">
 <segment>
-<wire x1="19" y1="9" x2="14.54" y2="9" width="0.1524" layer="91"/>
 <pinref part="+3V1" gate="G$1" pin="+3V3"/>
-<pinref part="X1" gate="G$1" pin="5"/>
-<wire x1="19" y1="9" x2="19" y2="8.46" width="0.1524" layer="91"/>
-<wire x1="19" y1="8.46" x2="20.38" y2="8.46" width="0.1524" layer="91"/>
+<wire x1="14.54" y1="9" x2="20" y2="9" width="0.1524" layer="91"/>
+<pinref part="X2" gate="G$1" pin="5"/>
+<wire x1="20" y1="9" x2="20" y2="8.46" width="0.1524" layer="91"/>
+<wire x1="20" y1="8.46" x2="20.38" y2="8.46" width="0.1524" layer="91"/>
 </segment>
 <segment>
@@
 <net name="N$2" class="0">
 <segment>
-<wire x1="-7" y1="14" x2="19" y2="14" width="0.1524" layer="91"/>
-<pinref part="X1" gate="G$1" pin="3"/>
-<wire x1="19" y1="14" x2="19" y2="13.54" width="0.1524" layer="91"/>
-<wire x1="19" y1="13.54" x2="20.38" y2="13.54" width="0.1524" layer="91"/>
+<wire x1="-7" y1="14" x2="20" y2="14" width="0.1524" layer="91"/>
 <pinref part="JOY1" gate="G$1" pin="Y"/>
 <wire x1="-7" y1="14" x2="-7" y2="13.5" width="0.1524" layer="91"/>
 <wire x1="-7" y1="13.5" x2="-10" y2="13.5" width="0.1524" layer="91"/>
+<pinref part="X2" gate="G$1" pin="3"/>
+<wire x1="20" y1="14" x2="20" y2="13.54" width="0.1524" layer="91"/>
+<wire x1="20" y1="13.54" x2="20.38" y2="13.54" width="0.1524" layer="91"/>
 </segment>
 </net>
@@
 <segment>
 <wire x1="-7" y1="17" x2="-4" y2="17" width="0.1524" layer="91"/>
-<pinref part="X1" gate="G$1" pin="2"/>
-<wire x1="-4" y1="17" x2="19" y2="17" width="0.1524" layer="91"/>
-<wire x1="19" y1="17" x2="19" y2="16.08" width="0.1524" layer="91"/>
-<wire x1="19" y1="16.08" x2="20.38" y2="16.08" width="0.1524" layer="91"/>
+<wire x1="-4" y1="17" x2="20" y2="17" width="0.1524" layer="91"/>
 <wire x1="-4" y1="17" x2="-4" y2="19.92" width="0.1524" layer="91"/>
 <junction x="-4" y="17"/>
@@
 <wire x1="-7" y1="16" x2="-10" y2="16" width="0.1524" layer="91"/>
 <pinref part="JOY1" gate="G$1" pin="SW"/>
+<pinref part="X2" gate="G$1" pin="2"/>
+<wire x1="20" y1="17" x2="20" y2="16.08" width="0.1524" layer="91"/>
+<wire x1="20" y1="16.08" x2="20.38" y2="16.08" width="0.1524" layer="91"/>
 </segment>
 </net>
@@
 <segment>
 <wire x1="16" y1="23.5" x2="16" y2="19" width="0.1524" layer="91"/>
-<wire x1="16" y1="19" x2="19" y2="19" width="0.1524" layer="91"/>
-<pinref part="X1" gate="G$1" pin="1"/>
-<wire x1="19" y1="19" x2="19" y2="18.62" width="0.1524" layer="91"/>
-<wire x1="19" y1="18.62" x2="20.38" y2="18.62" width="0.1524" layer="91"/>
+<wire x1="16" y1="19" x2="20" y2="19" width="0.1524" layer="91"/>
 <pinref part="POT1" gate="G$1" pin="P$3"/>
+<pinref part="X2" gate="G$1" pin="1"/>
+<wire x1="20" y1="19" x2="20" y2="18.62" width="0.1524" layer="91"/>
+<wire x1="20" y1="18.62" x2="20.38" y2="18.62" width="0.1524" layer="91"/>
 </segment>
 </net>
@@
 <segment>
 <wire x1="-10" y1="11" x2="20.38" y2="11" width="0.1524" layer="91"/>
-<pinref part="X1" gate="G$1" pin="4"/>
 <pinref part="JOY1" gate="G$1" pin="X"/>
-</segment>
-</net>
+<pinref part="X2" gate="G$1" pin="4"/>
+</segment>
+</net>
+<net name="+9V" class="0">
+<segment>
+<wire x1="20" y1="6" x2="14.54" y2="6" width="0.1524" layer="91"/>
+<pinref part="SUPPLY5" gate="G$1" pin="+9V"/>
+<pinref part="X2" gate="G$1" pin="6"/>
+<wire x1="20" y1="6" x2="20" y2="5.92" width="0.1524" layer="91"/>
+<wire x1="20" y1="5.92" x2="20.38" y2="5.92" width="0.1524" layer="91"/>
+</segment>
+<segment>
+<wire x1="-30.54" y1="34" x2="-34" y2="34" width="0.1524" layer="91"/>
+<pinref part="X1" gate="G$1" pin="1"/>
+<wire x1="-34" y1="34" x2="-34" y2="34.46" width="0.1524" layer="91"/>
+<wire x1="-34" y1="34.46" x2="-35.38" y2="34.46" width="0.1524" layer="91"/>
+<pinref part="SUPPLY6" gate="G$1" pin="+9V"/>
+</segment>
+</net>
