File: SuniderPra/SuniderPra.brd (EAGLE design)
At the start: 100 x 80 mm, 16 parts, among them Q1 2SK4017(Q), Q2 2SK4017(Q), U1 GY-521MPU6050, X1 B2P-VH, X2 B2P-VH, X3 B2P-VH

Commit message: Add files via upload
Parts:
- removed JP3: (no value), pinhead:1X04
- removed Q1, Q2: 2SK4017(Q), 2SK4017_Q_:TO230P230X650X740-3P
- removed U1: GY-521MPU6050, MPU6050:GY-521
- added C3: 0.1u, rcl:C050-024X044
- added F1: MF-R300, MF-R300:MFR300
- added FET_DC1, FET_DC2: 2SK4017(Q), 2SK4017_Q_:TO230P230X650X740-3P
- added IC1: TD62083APG_O,N_, SamacSys_Parts:DIP762W60P254L2510H445Q18N
- added IMU: GY-521MPU6050, MPU6050:GY-521
- added LED1, LED2, LED3, LED4: (no value), led:LED3MM
- added R5, R6, R7, R8: led, rcl:0207/7
- added SERVO1, SERVO2: B3B-XH-2, con-JST XH:B3B-XH-A
- added X4: B2PS-VH, con-JST VH:B2PS-VH
- JP1, JP2: device pinhead:1X03 -> pinhead:1X06
- R1, R3: value 1k -> 100
- R2, R4: value 1k -> 10k
- X1: value B2P-VH -> B6B-XH-2; device con-JST VH:B2P-VH -> con-JST XH:B6B-XH-A
- X2, X3: value B2P-VH -> B2PS-VH; device con-JST VH:B2P-VH -> con-JST VH:B2PS-VH
- moved C2 174.1 mm to (68.0, 56.0), turned to 270 degrees
- moved C1 155.0 mm to (73.2, 29.0), turned to 90 degrees
- moved X3 118.2 mm to (19.0, 19.0)
- moved X1 117.4 mm to (34.0, 60.0)
- moved R3 115.9 mm to (15.6, 41.2), turned to 180 degrees
- moved X2 110.1 mm to (12.0, 47.0), turned to 180 degrees
- moved R4 107.3 mm to (6.40, 31.9), turned to 180 degrees
- moved JP2 86.6 mm to (35.0, 11.0)
- moved JP1 84.3 mm to (35.0, 3.00)
- moved R2 78.8 mm to (6.50, 35.9)
- moved R1 78.2 mm to (3.00, 43.4), turned to 270 degrees
- moved A1 64.2 mm to (54.0, 34.0)
Connections:
- new net JOYSW: A1.3.10, X1.2
- new net LED1: A1.4.9, R5.1
- new net LED2: A1.4.10, R6.1
- new net LED3: A1.4.15, R7.1
- new net N$10: FET_DC1.2, X4.2
- new net N$12: IC1.13, JP1.4
- new net N$13: A1.3.1, R1.1
- new net N$14: LED1.A, R5.2
- new net N$15: LED3.A, R7.2
- new net N$16: IC1.14, JP1.3
- new net N$17: IC1.15, JP2.3
- new net N$18: A1.4.6, X1.1
- new net N$19: F1.1, X2.1
- new net N$20: A1.4.7, X1.3
- new net N$21: LED4.A, R8.2
- new net N$22: IC1.16, JP2.4
- new net N$23: IC1.17, JP2.5
- new net N$24: IC1.18, JP2.6
- new net PHOTO1: A1.4.11, SERVO2.1
- new net PHOTO2: A1.4.12, SERVO1.1
- new net STEP11: A1.3.12, IC1.4
- new net STEP12: A1.3.13, IC1.3
- new net STEP13: A1.3.14, IC1.2
- new net STEP14: A1.3.15, IC1.1
- new net STEP21: A1.3.5, IC1.8
- new net STEP22: A1.3.6, IC1.7
- new net STEP23: A1.3.9, IC1.6
- new net STEP24: A1.3.11, IC1.5
- net +3V3: now also IMU.VCC, SERVO1.2, SERVO2.2, X1.5; no longer JP3.1, U1.VCC
- net +9V: now also C3.2, F1.2, IC1.10, JP1.1, JP2.1, R8.1, X4.1; no longer Q1.2, Q2.2, X1.1, X2.1
- net GND: now also C3.1, FET_DC1.3, FET_DC2.3, IC1.9, IMU.GND, LED1.K, LED2.K, LED3.K, LED4.K, SERVO1.3, SERVO2.3, X1.6; no longer JP1.1, JP2.1, JP3.2, Q1.3, Q2.3, U1.GND, X1.2, X3.2
- net N$1: now also IMU.SCL; no longer U1.SCL
- net N$11: now also LED2.A, R6.2; no longer A1.4.10, R3.1
- net N$2: now also IMU.SDA; no longer U1.SDA
- net N$3: now also IC1.11, JP1.6; no longer A1.3.13, JP1.3
- net N$4: now also IC1.12, JP1.5; no longer A1.3.12, JP2.3
- net N$5: now also A1.4.8, X1.4; no longer A1.4.9, R1.1
- net N$6: now also FET_DC1.1; no longer Q1.1
- net N$7: now also FET_DC2.2, X3.2; no longer A1.4.6, JP3.4
- net N$8: now also A1.3.2, R3.1; no longer A1.4.5, JP3.3
- net N$9: now also FET_DC2.1; no longer Q2.1
Routing:
- net +9V: track 0.00 -> 265.1 mm
- net GND: track 0.00 -> 249.5 mm
- net +3V3: track 0.00 -> 124.5 mm, vias 0 -> 1
- net N$3: track 0.00 -> 53.8 mm
- net JOYSW: track 0.00 -> 53.6 mm, vias 0 -> 1
- net N$4: track 0.00 -> 50.5 mm
- net N$12: track 0.00 -> 47.3 mm
- net N$13: track 0.00 -> 47.1 mm, vias 0 -> 2
- net N$5: track 0.00 -> 47.0 mm
- net N$10: track 0.00 -> 44.5 mm
- net N$16: track 0.00 -> 44.4 mm
- net N$20: track 0.00 -> 43.4 mm
- net N$18: track 0.00 -> 38.8 mm
- net N$2: track 0.00 -> 34.8 mm
- net N$1: track 0.00 -> 34.7 mm
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- added copper zone on layer 16, net GND
Other:
- board size 100 x 80 mm -> 80 x 65 mm

Commit message: Add files via upload
Parts:
- removed F1: MF-R300, MF-R300:MFR300
- removed JP1, JP2: (no value), pinhead:1X06
- added LED6: (no value), led:LED3MM
- added R10: led, rcl:0207/7
- added R11, R13: 220, rcl:0207/7
- added R12, R14: 10k, rcl:0207/7
- added X5: B2B-XH-2, con-JST XH:B2B-XH-A
- added X6: B2PS-VH, con-JST VH:B2PS-VH
- added X7, X8: B6B-XH-2, con-JST XH:B6B-XH-A
- R1, R3: value 100 -> 470
- moved LED1 37.9 mm to (41.0, 11.0)
- moved LED2 31.6 mm to (46.0, 11.0)
- moved LED3 26.0 mm to (51.0, 11.0)
- moved IMU 22.6 mm to (47.0, 33.0)
- moved C1 21.2 mm to (54.0, 20.0), turned to 180 degrees
- moved SERVO1 21.0 mm to (47.5, 3.40)
- moved R3 17.7 mm to (28.8, 29.4)
- moved LED4 17.5 mm to (12.0, 29.0)
- moved A1 16.0 mm to (70.0, 35.0)
- moved C3 15.5 mm to (45.0, 48.0), turned to 180 degrees
- moved X1 15.0 mm to (49.0, 60.0)
- moved R4 13.6 mm to (20.0, 31.1)
- moved R1 12.0 mm to (15.0, 43.4)
- moved R8 11.5 mm to (13.9, 33.9), turned to 180 degrees
- moved SERVO2 8.46 mm to (63.0, 3.40)
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Connections:
- removed net N$19: F1.1, X2.1
- removed net N$24: IC1.18, JP2.6
- new net +5V/1: R8.1, X2.1, X3.1, X4.1, X6.1
- new net N$25: LED6.A, R10.2
- new net N$26: R13.1, SERVO2.3
- new net N$27: R11.1, SERVO1.3
- new net N$28: IC1.11, X8.4
- net +9V: now also R10.1, X5.1, X7.5, X7.6, X8.5, X8.6; no longer F1.2, JP1.1, JP1.2, JP2.1, JP2.2, R8.1, X3.1, X4.1
- net GND: now also LED6.K, R11.2, R12.2, R13.2, R14.2, X5.2, X6.2; no longer SERVO1.3, SERVO2.3
- net N$12: now also X8.2; no longer JP1.4
- net N$16: now also X8.1; no longer JP1.3
- net N$17: now also X7.4; no longer JP2.3
- net N$22: now also X7.3; no longer JP2.4
- net N$23: now also X7.2; no longer JP2.5
- net N$3: now also IC1.18, X7.1; no longer IC1.11, JP1.6
- net N$4: now also X8.3; no longer JP1.5
- net PHOTO1: now also R12.1, SERVO1.1; no longer SERVO2.1
- net PHOTO2: now also R14.1, SERVO2.1; no longer SERVO1.1
- net STEP21: now also A1.3.11, IC1.5; no longer A1.3.5, IC1.8
- net STEP22: now also A1.3.9, IC1.6; no longer A1.3.6, IC1.7
- net STEP23: now also A1.3.6, IC1.7; no longer A1.3.9, IC1.6
- net STEP24: now also A1.3.5, IC1.8; no longer A1.3.11, IC1.5
Routing:
- net +5V/1: track 0.00 -> 163.7 mm
- net +9V: track 265.1 -> 129.7 mm
- net N$4: track 50.5 -> 8.47 mm
- net N$12: track 47.3 -> 8.48 mm
- net N$3: track 53.8 -> 15.7 mm
- net N$16: track 44.4 -> 8.50 mm
- net N$10: track 44.5 -> 11.1 mm
- net N$19: track 28.0 -> 0.00 mm
- net PHOTO1: track 27.8 -> 54.5 mm
- net N$2: track 34.8 -> 9.37 mm
- net N$1: track 34.7 -> 9.79 mm
- net STEP22: track 5.64 -> 30.5 mm
- net N$11: track 2.91 -> 23.8 mm
- net STEP21: track 5.57 -> 24.5 mm, vias 0 -> 1
- net N$14: track 9.36 -> 28.2 mm
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Other:
- board text added: "210315"

Commit message: Add files via upload
Parts:
- removed X1: B6B-XH-2, con-JST XH:B6B-XH-A
- removed X5: B2B-XH-2, con-JST XH:B2B-XH-A
- added X9: B7B-XH-2, con-JST XH:B7B-XH-A
- renumbered SERVO2 to PHOTO2
Connections:
- removed net N$20: A1.4.7, X1.3
- new net N$19: A1.4.7, X9.3
- net +3V3: now also X9.5; no longer X1.5
- net +9V: now also X9.6; no longer X5.1
- net GND: now also X9.7; no longer X1.6, X5.2
- net JOYSW: now also X9.2; no longer X1.2
- net N$18: now also X9.1; no longer X1.1
- net N$5: now also X9.4; no longer X1.4
Routing:
- net N$19: track 0.00 -> 50.9 mm
- net N$20: track 44.1 -> 0.00 mm
- net GND: track 242.1 -> 278.9 mm, vias 0 -> 4
- net N$18: track 36.7 -> 44.4 mm
- net N$5: track 47.7 -> 54.4 mm
- net JOYSW: track 42.4 -> 49.1 mm
- net +3V3: track 142.3 -> 148.2 mm
- net +9V: track 129.7 -> 125.1 mm
- net +5V/1: vias 0 -> 5
Other:
- board text added: "3V"
- board text added: "9V"
- board text added: "G"
- board text added: "G + sig"
- board text added: "Jx"
- board text added: "Jy"
- board text added: "PHOTO1"
- board text added: "Sw"
- board text added: "USB"
- board text added: "Vol"
