File: PhasedArray3/PhasedArray3.sch (EAGLE design)
At the start: 31 parts, among them IC1 NJU7034M, IC2 NJM7805FA, U1 NJM7905FA-ND, X1 B2B-XH-2, X2 B2B-XH-2

Commit message: Add files via upload
Parts:
- removed JP1: (no value), pinhead:PINHD-1X2
- added C16, C20, C26, C30, C36, C40: 1n, rcl:C-EUC0603K
- added C17, C27, C37: 10p, rcl:C-EUC0603K
- added C18, C19, C28, C29, C38, C39: 330p, rcl:C-EUC0603K
- added C21, C31, C41: 15p, rcl:C-EUC0603K
- added C22, C24, C32, C34, C42, C44: 100n, rcl:C-EUC0603K
- added C23, C25, C33, C35, C43, C45: 10n, rcl:C-EUC0603K
- added IC3, IC4, IC5: NJU7034M, SamacSys_Parts:NJU7034M
- added R10, R19, R28: 3.9k, rcl:R-EU_R0603
- added R11, R20, R29: 1k, rcl:R-EU_R0603
- added R12, R21, R30: 10k, rcl:R-EU_R0603
- added R13, R22, R31: 160k, rcl:R-EU_R0603
- added R14, R23, R32: 5.1k, rcl:R-EU_R0603
- added R15, R24, R33: 2.7k, rcl:R-EU_R0603
- added R16, R25, R34: 82k, rcl:R-EU_R0603
- added R17, R26, R35: 15k, rcl:R-EU_R0603
- added R18, R27, R36: 100k, rcl:R-EU_R0603
- added VR2, VR3, VR4: 3361P-1-504GLF, 3361P-1-504GLF:3361P-1-504GLF
- added X3: S8B-XH-A, con-JST XH:S8B-XH-A
- added X4, X5, X6, X7: S2B-XH-A, con-JST XH:S2B-XH-A
- X1, X2: value B2B-XH-2 -> S2B-XH-A; device con-JST XH:B2B-XH-2 -> con-JST XH:S2B-XH-A
Connections:
- removed net N$9: C6.1, IC1.OUT3, R9.1
- new net AO1+: C41.1, IC5.OUT3, R36.1, X3.8
- new net AO2+: C31.1, IC4.OUT3, R27.1, X3.6
- new net AO3+: C21.1, IC3.OUT3, R18.1, X3.4
- new net AO4+: C6.1, IC1.OUT3, R9.1, X3.2
- new net N$13: IC1.IN-2, IC1.OUT2
- new net N$14: R10.2, R11.2, X2.1
- new net N$15: C16.1, R11.1
- new net N$16: C16.2, R12.2
- new net N$17: C17.1, IC3.IN-1, R12.1, R13.2
- new net N$18: C17.2, IC3.OUT1, R13.1, R14.1
- new net N$19: C18.1, C19.1, R14.2, R15.1
- new net N$20: C18.2, IC3.IN-4, R16.1
- new net N$21: C19.2, C20.1, IC3.OUT4, R16.2
- new net N$22: C21.2, IC3.IN-3, R17.2, R18.2
- new net N$24: C20.2, VR2.CCW
- new net N$25: R17.1, VR2.2, VR2.CW
- new net N$26: IC3.IN-2, IC3.OUT2
- new net N$27: R19.2, R20.2, X6.1
- new net N$28: C26.1, R20.1
- new net N$29: C26.2, R21.2
- new net N$30: C27.1, IC4.IN-1, R21.1, R22.2
- new net N$31: C27.2, IC4.OUT1, R22.1, R23.1
- new net N$32: C28.1, C29.1, R23.2, R24.1
- new net N$33: C28.2, IC4.IN-4, R25.1
- new net N$34: C29.2, C30.1, IC4.OUT4, R25.2
- new net N$35: C31.2, IC4.IN-3, R26.2, R27.2
- new net N$37: C30.2, VR3.CCW
- new net N$38: R26.1, VR3.2, VR3.CW
- new net N$39: IC4.IN-2, IC4.OUT2
- new net N$40: R28.2, R29.2, X7.1
- new net N$41: C36.1, R29.1
- new net N$42: C36.2, R30.2
- new net N$43: C37.1, IC5.IN-1, R30.1, R31.2
- new net N$44: C37.2, IC5.OUT1, R31.1, R32.1
- new net N$45: C38.1, C39.1, R32.2, R33.1
- new net N$46: C38.2, IC5.IN-4, R34.1
- new net N$47: C39.2, C40.1, IC5.OUT4, R34.2
- new net N$48: C41.2, IC5.IN-3, R35.2, R36.2
- new net N$50: C40.2, VR4.CCW
- new net N$51: R35.1, VR4.2, VR4.CW
- new net N$52: IC5.IN-2, IC5.OUT2
- net +5V: now also C22.1, C23.1, C32.1, C33.1, C42.1, C43.1, IC3.VDD, IC4.VDD, IC5.VDD
- net +9V: now also X4.1; no longer X1.2
- net -5V: now also C24.1, C25.1, C34.1, C35.1, C44.1, C45.1, IC3.VSS, IC4.VSS, IC5.VSS
- net -9V: now also X5.2; no longer X2.1
- net GND: now also C22.2, C23.2, C24.2, C25.2, C32.2, C33.2, C34.2, C35.2, C42.2, C43.2, C44.2, C45.2, IC1.IN+2, IC3.IN+1, IC3.IN+2, IC3.IN+3, IC3.IN+4, IC4.IN+1, IC4.IN+2, IC4.IN+3, IC4.IN+4, IC5.IN+1, IC5.IN+2, IC5.IN+3, IC5.IN+4, R10.1, R15.2, R19.1, R24.2, R28.1, R33.2, X1.2, X3.1, X3.3, X3.5, X3.7, X4.2, X5.1, X6.2, X7.2; no longer JP1.1, X1.1
- net N$1: now also X1.1; no longer JP1.2
Other:
- moved on the sheet: C5, X1, X2
